File: stepper_driver.sch (EAGLE design)
At the start: 12 parts, among them IC1 L293D, IC2 L293D, Q1 IRLML5203, Q2 IRLML5203

Commit message: Polishing artwork
Parts:
- added C1, C2: (no value), rcl:C-USC1206
- added LED1: (no value), led:LED5MM
- added R3, R4, R5: 1k, rcl:R-US_0207/10
- R1, R2: value (none) -> 10k
Connections:
- new net N$10: LED1.C, R3.2
- new net N$12: Q1.D, R1.2, R5.2
- new net N$13: Q2.D, R2.2, R4.1
- net 5V: now also C1.1, C2.1, LED1.A
- net GND: now also C1.2, C2.2, R3.1
- net N$5: now also R5.1; no longer Q1.D, R1.2
- net N$7: now also R4.2; no longer Q2.D, R2.2
Changed lines of the file:
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@@
 <part name="GND6" library="SparkFun" deviceset="GND" device=""/>
 <part name="P+3" library="SparkFun" deviceset="VCC" device=""/>
-<part name="R1" library="rcl" deviceset="R-US_" device="0207/10"/>
-<part name="R2" library="rcl" deviceset="R-US_" device="0207/10"/>
+<part name="R1" library="rcl" deviceset="R-US_" device="0207/10" value="10k"/>
+<part name="R2" library="rcl" deviceset="R-US_" device="0207/10" value="10k"/>
 <part name="GND7" library="SparkFun" deviceset="GND" device=""/>
 <part name="GND8" library="SparkFun" deviceset="GND" device=""/>
+<part name="R3" library="rcl" deviceset="R-US_" device="0207/10" value="1k"/>
+<part name="GND9" library="SparkFun" deviceset="GND" device=""/>
+<part name="LED1" library="led" deviceset="LED" device="5MM"/>
+<part name="U$10" library="SparkFun" deviceset="5V" device=""/>
+<part name="C1" library="rcl" deviceset="C-US" device="C1206"/>
+<part name="C2" library="rcl" deviceset="C-US" device="C1206"/>
+<part name="GND10" library="SparkFun" deviceset="GND" device=""/>
+<part name="GND11" library="SparkFun" deviceset="GND" device=""/>
+<part name="U$11" library="SparkFun" deviceset="5V" device=""/>
+<part name="U$12" library="SparkFun" deviceset="5V" device=""/>
+<part name="R4" library="rcl" deviceset="R-US_" device="0207/10" value="1k"/>
+<part name="R5" library="rcl" deviceset="R-US_" device="0207/10" value="1k"/>
 </parts>
 <sheets>
@@
 <instance part="GND7" gate="1" x="20.32" y="86.36"/>
 <instance part="GND8" gate="1" x="119.38" y="86.36"/>
+<instance part="R3" gate="G$1" x="144.78" y="91.44" rot="R90"/>
+<instance part="GND9" gate="1" x="144.78" y="83.82"/>
+<instance part="LED1" gate="G$1" x="144.78" y="101.6"/>
+<instance part="U$10" gate="G$1" x="144.78" y="104.14"/>
+<instance part="C1" gate="G$1" x="157.48" y="91.44"/>
+<instance part="C2" gate="G$1" x="165.1" y="91.44"/>
+<instance part="GND10" gate="1" x="157.48" y="83.82"/>
+<instance part="GND11" gate="1" x="165.1" y="83.82"/>
+<instance part="U$11" gate="G$1" x="157.48" y="93.98"/>
+<instance part="U$12" gate="G$1" x="165.1" y="93.98"/>
+<instance part="R4" gate="G$1" x="111.76" y="99.06" rot="R180"/>
+<instance part="R5" gate="G$1" x="27.94" y="99.06" rot="R180"/>
 </instances>
 <busses>
@@
 <pinref part="GND8" gate="1" pin="GND"/>
 </segment>
+<segment>
+<pinref part="R3" gate="G$1" pin="1"/>
+<pinref part="GND9" gate="1" pin="GND"/>
+</segment>
+<segment>
+<pinref part="C1" gate="G$1" pin="2"/>
+<pinref part="GND10" gate="1" pin="GND"/>
+</segment>
+<segment>
+<pinref part="C2" gate="G$1" pin="2"/>
+<pinref part="GND11" gate="1" pin="GND"/>
+</segment>
 </net>
 <net name="N$5" class="0">
@@
 <pinref part="IC1" gate="G$1" pin="2A"/>
 <wire x1="50.8" y1="99.06" x2="33.02" y2="99.06" width="0.1524" layer="91"/>
-<pinref part="Q1" gate="G$1" pin="D"/>
-<pinref part="R1" gate="G$1" pin="2"/>
-<junction x="20.32" y="99.06"/>
 <pinref part="IC2" gate="G$1" pin="2A"/>
-<wire x1="33.02" y1="99.06" x2="20.32" y2="99.06" width="0.1524" layer="91"/>
 <wire x1="33.02" y1="99.06" x2="33.02" y2="33.02" width="0.1524" layer="91"/>
 <wire x1="33.02" y1="33.02" x2="50.8" y2="33.02" width="0.1524" layer="91"/>
+<pinref part="R5" gate="G$1" pin="1"/>
 <junction x="33.02" y="99.06"/>
 </segment>
@@
 <segment>
 <pinref part="IC1" gate="G$1" pin="3A"/>
-<wire x1="81.28" y1="99.06" x2="114.3" y2="99.06" width="0.1524" layer="91"/>
-<pinref part="Q2" gate="G$1" pin="D"/>
-<pinref part="R2" gate="G$1" pin="2"/>
-<junction x="119.38" y="99.06"/>
+<wire x1="81.28" y1="99.06" x2="106.68" y2="99.06" width="0.1524" layer="91"/>
 <pinref part="IC2" gate="G$1" pin="3A"/>
-<wire x1="114.3" y1="99.06" x2="119.38" y2="99.06" width="0.1524" layer="91"/>
-<wire x1="114.3" y1="99.06" x2="114.3" y2="33.02" width="0.1524" layer="91"/>
-<wire x1="114.3" y1="33.02" x2="81.28" y2="33.02" width="0.1524" layer="91"/>
-<junction x="114.3" y="99.06"/>
+<wire x1="106.68" y1="99.06" x2="106.68" y2="33.02" width="0.1524" layer="91"/>
+<wire x1="106.68" y1="33.02" x2="81.28" y2="33.02" width="0.1524" layer="91"/>
+<pinref part="R4" gate="G$1" pin="2"/>
+<junction x="106.68" y="99.06"/>
 </segment>
 </net>
@@
 <wire x1="83.82" y1="63.5" x2="81.28" y2="63.5" width="0.1524" layer="91"/>
 </segment>
+<segment>
+<pinref part="LED1" gate="G$1" pin="A"/>
+<pinref part="U$10" gate="G$1" pin="5V"/>
+</segment>
+<segment>
+<pinref part="C1" gate="G$1" pin="1"/>
+<pinref part="U$11" gate="G$1" pin="5V"/>
+</segment>
+<segment>
+<pinref part="C2" gate="G$1" pin="1"/>
+<pinref part="U$12" gate="G$1" pin="5V"/>
+</segment>
 </net>
 <net name="VCC" class="0">
@@
 </segment>
 </net>
+<net name="N$10" class="0">
+<segment>
+<pinref part="R3" gate="G$1" pin="2"/>
+<pinref part="LED1" gate="G$1" pin="C"/>
+</segment>
+</net>
+<net name="N$12" class="0">
+<segment>
+<pinref part="Q1" gate="G$1" pin="D"/>
+<pinref part="R1" gate="G$1" pin="2"/>
+<pinref part="R5" gate="G$1" pin="2"/>
+<wire x1="22.86" y1="99.06" x2="20.32" y2="99.06" width="0.1524" layer="91"/>
+<junction x="20.32" y="99.06"/>
+</segment>
+</net>
+<net name="N$13" class="0">
+<segment>
+<pinref part="Q2" gate="G$1" pin="D"/>
+<pinref part="R2" gate="G$1" pin="2"/>
+<pinref part="R4" gate="G$1" pin="1"/>
+<wire x1="116.84" y1="99.06" x2="119.38" y2="99.06" width="0.1524" layer="91"/>
+<junction x="119.38" y="99.06"/>
+</segment>
+</net>

Commit message: Fix to only for single L293D IC
Parts:
- removed C1: (no value), rcl:C-USC1206
- removed IC2: L293D, st-microelectronics:L293D
- removed JP1: (no value), pinhead:PINHD-1X4
- added D1: 1N4004, diode:1N4004
- added JP7: (no value), pinhead:PINHD-1X2
- JP6: device pinhead:PINHD-1X4 -> pinhead:PINHD-1X2
Connections:
- removed net N$11: IC2.4Y, JP6.1
- removed net N$8: IC2.2Y, JP6.3
- removed net N$9: IC2.3Y, JP6.2
- net 5V: no longer C1.1, IC2.VCC1
- net GND: no longer C1.2, IC2.GND1, IC2.GND2, IC2.GND3, IC2.GND4
- net IC2_EN: no longer IC2.1-2EN, IC2.3-4EN
- net N$1: now also JP6.2; no longer JP1.4
- net N$2: now also JP6.1; no longer JP1.3
- net N$3: now also JP7.2; no longer JP1.2
- net N$4: now also JP7.1; no longer JP1.1
- net N$5: no longer IC2.2A
- net N$6: now also D1.C, IC1.VCC2; no longer IC2.1Y, JP6.4
- net N$7: no longer IC2.3A
- net S1: no longer IC2.1A
- net S2: no longer IC2.4A
- net VCC: now also D1.A; no longer IC1.VCC2, IC2.VCC2
